Commit message: Added new controllers

File: 01-kuka-mobile-base/iiwa7.urdf (robot description, URDF)
Before this commit: robot kuka_iiwa, 8 links, 7 joints
Links:
- added link gripper1, mass 0.2; collision box size=0.03 0.01 0.07; visual box size=0.03 0.01 0.07
- added link gripper2, mass 0.2; collision box size=0.03 0.01 0.07; visual box size=0.03 0.01 0.07
- added link ground, mass 0.0001
- added link virtual1, mass 0.0001
- added link virtual2, mass 0.0001
- link base_link: geometry visual box size=0.4 0.7 0.25; visual mesh filename=../../../robot_models/iiwa7/meshes/base.obj scale=1 1 1
- link link1: geometry visual mesh filename=../../../robot_models/iiwa7/meshes/link0.obj scale=1 1 1
- link link2: geometry visual mesh filename=../../../robot_models/iiwa7/meshes/link1.obj scale=1 1 1
- link link3: geometry visual mesh filename=../../../robot_models/iiwa7/meshes/link2.obj scale=1 1 1
- link link4: geometry visual mesh filename=../../../robot_models/iiwa7/meshes/link3.obj scale=1 1 1
- link link5: geometry visual mesh filename=../../../robot_models/iiwa7/meshes/link4.obj scale=1 1 1
- link link6: geometry visual mesh filename=../../../robot_models/iiwa7/meshes/link5.obj scale=1 1 1
- link link7: geometry visual mesh filename=../../../robot_models/iiwa7/meshes/link6.obj scale=1 1 1
Joints:
- added joint jgripper1: type prismatic, parent link7, child gripper1, origin xyz=0 0 0.07 rpy=0.000000 0.000000 0.000000, axis 0 1 0, limit lower=-3.0543 upper=3.0543 effort=40 velocity=3.1416
- added joint jgripper2: type prismatic, parent link7, child gripper2, origin xyz=0 0 0.07 rpy=0.000000 0.000000 3.1415926535897, axis 0 1 0, limit lower=-3.0543 upper=3.0543 effort=40 velocity=3.1416
- added joint jpx: type prismatic, parent ground, child virtual1, origin xyz=0 0 0 rpy=0 0 0, axis 1 0 0, limit lower=-2.967 upper=2.967 effort=176 velocity=1.7104
- added joint jpy: type prismatic, parent virtual1, child virtual2, origin xyz=0 0 0 rpy=0 0 0, axis 0 1 0, limit lower=-2.967 upper=2.967 effort=176 velocity=1.7104
- added joint jr: type revolute, parent virtual2, child base_link, origin xyz=0 0 0.35 rpy=0 0 0, axis 0 0 1, limit lower=-2.967 upper=2.967 effort=176 velocity=1.7104
