Commit message: Added controllers

File: 02-kuka-dual-arm/iiwa7.urdf (robot description, URDF)
Before this commit: robot kuka_iiwa, 13 links, 12 joints
Links:
- added link arm2_gripper1, mass 0.2; collision box size=0.03 0.01 0.07; visual box size=0.03 0.01 0.07
- added link arm2_gripper2, mass 0.2; collision box size=0.03 0.01 0.07; visual box size=0.03 0.01 0.07
- added link arm2_link1, mass 3.4525; visual mesh filename=../../../robot_models/iiwa7/meshes/link0.obj scale=1 1 1
- added link arm2_link2, mass 3.4821; visual mesh filename=../../../robot_models/iiwa7/meshes/link1.obj scale=1 1 1
- added link arm2_link3, mass 4.05623; visual mesh filename=../../../robot_models/iiwa7/meshes/link2.obj scale=1 1 1
- added link arm2_link4, mass 3.4822; visual mesh filename=../../../robot_models/iiwa7/meshes/link3.obj scale=1 1 1
- added link arm2_link5, mass 2.1633; visual mesh filename=../../../robot_models/iiwa7/meshes/link4.obj scale=1 1 1
- added link arm2_link6, mass 2.3466; visual mesh filename=../../../robot_models/iiwa7/meshes/link5.obj scale=1 1 1
- added link arm2_link7, mass 3.529; visual mesh filename=../../../robot_models/iiwa7/meshes/link6.obj scale=1 1 1
- link base_link: geometry visual box size=0.4 0.7 0.25; visual mesh filename=../../../robot_models/iiwa7/meshes/base.obj scale=1 1 1
- link gripper1: geometry collision box size=0.03 0.01 0.07; visual box size=0.03 0.01 0.07
Joints:
- added joint arm2_j0: type revolute, parent base_link, child arm2_link1, origin xyz=0.23 -0.2 0.375 rpy=0 -1.047197 3.141592, axis 0 0 1, limit lower=-2.967 upper=2.967 effort=176 velocity=1.7104
- added joint arm2_j1: type revolute, parent arm2_link1, child arm2_link2, origin xyz=0.000000 0.000000 0.19 rpy=0.000000 0.000000 0.000000, axis 0 1 0, limit lower=-2.0944 upper=2.0944 effort=176 velocity=1.7104
- added joint arm2_j2: type revolute, parent arm2_link2, child arm2_link3, origin xyz=0.000000 0.000000 0.21 rpy=0.000000 0.000000 0.000000, axis 0 0 1, limit lower=-2.967 upper=2.967 effort=110 velocity=1.7453
- added joint arm2_j3: type revolute, parent arm2_link3, child arm2_link4, origin xyz=0.000000 0.000000 0.19 rpy=0.000000 0.000000 3.1415926535897, axis 0 1 0, limit lower=-2.0944 upper=2.0944 effort=110 velocity=2.2689
- added joint arm2_j4: type revolute, parent arm2_link4, child arm2_link5, origin xyz=0.000000 0.000000 0.21 rpy=0.000000 0.000000 -3.1415926535897, axis 0 0 1, limit lower=-2.967 upper=2.967 effort=110 velocity=2.4434
- added joint arm2_j5: type revolute, parent arm2_link5, child arm2_link6, origin xyz=0.000000 -0.06070 0.19 rpy=0.000000 0.000000 0.000000, axis 0 1 0, limit lower=-2.0944 upper=2.0944 effort=40 velocity=3.1416
- added joint arm2_j6: type revolute, parent arm2_link6, child arm2_link7, origin xyz=0.000000 0.06070 0.081000 rpy=0.000000 0.000000 0.000000, axis 0 0 1, limit lower=-3.0543 upper=3.0543 effort=40 velocity=3.1416
- added joint arm2_jgripper1: type prismatic, parent arm2_link7, child arm2_gripper1, origin xyz=0 0 0.07 rpy=0.000000 0.000000 0.000000, axis 0 1 0, limit lower=-3.0543 upper=3.0543 effort=40 velocity=3.1416
- added joint arm2_jgripper2: type prismatic, parent arm2_link7, child arm2_gripper2, origin xyz=0 0 0.07 rpy=0.000000 0.000000 3.1415926535897, axis 0 1 0, limit lower=-3.0543 upper=3.0543 effort=40 velocity=3.1416
- joint j0: origin xyz=0 -0.2 0.15 rpy=0 0 0 -> xyz=-0.23 -0.2 0.375 rpy=0 -1.047197 0

File: robot_models/robotObject/robotObject.urdf (robot description, URDF)
Before this commit: robot robotObject, 7 links, 6 joints
Links:
- removed link virtual4
- removed link virtual5
- link base_link: mass 0.1 -> 5; geometry visual box size=0.1 0.1 0.1; visual box size=0.4 0.7 0.25
Joints:
- removed joint jrx
- removed joint jry
- removed joint jrz
- added joint jr: type revolute, parent virtual3, child base_link, origin xyz=0 0 0.35 rpy=0 0 0, axis 0 0 1, limit lower=-2.967 upper=2.967 effort=176 velocity=1.7104
